File: Eagle Files/Board v1.brd (EAGLE design)
At the start: 150 x 37 mm, 9 parts

Commit message: Modified schematic and board for 16/12 and 16/8/4 pin connector setups.
Parts:
- removed J3: (no value), pinhead:1X08
- added JP1: (no value), pinhead:1X12
- moved J4 0.51 mm to (73.7, 33.0)
Connections:
- net N$31 renamed RST
- removed net +5V: J8.2, U$1.+5V, U$1.5V
- removed net N$20: R1.1, U$1.B6
- removed net N$21: R2.1, U$1.B5
- removed net N$22: R3.1, U$1.B4
- new net B4: JP1.12, R3.1, U$1.B4
- new net B5: JP1.11, R2.1, U$1.B5
- new net B6: JP1.9, R1.1, U$1.B6
- new net N$30: JP1.1, U$1.F1
- new net VCC: J8.2, JP1.10, U$1.+5V, U$1.5V
- net N$23: now also JP1.8; no longer J3.8
- net N$24: now also JP1.7; no longer J3.7
- net N$25: now also JP1.6; no longer J3.6
- net N$26: now also JP1.5; no longer J3.5
- net N$27: now also JP1.4; no longer J3.3
- net N$28: now also JP1.3, U$1.E6; no longer J3.1, U$1.F0
- net N$29: now also JP1.2, U$1.F0; no longer J3.2, U$1.E6
Routing:
- net VCC: track 0.00 -> 115.4 mm
- net +5V: track 110.7 -> 0.00 mm
- net GND: track 90.8 -> 0.00 mm
- net B5: track 0.00 -> 68.6 mm
- net B4: track 0.00 -> 65.8 mm, vias 0 -> 1
- net N$30: track 0.00 -> 64.9 mm
- net B6: track 0.00 -> 61.7 mm
- net N$22: track 53.8 -> 0.00 mm
- net N$21: track 49.6 -> 0.00 mm
- net N$20: track 45.5 -> 0.00 mm
- net N$27: track 67.8 -> 56.6 mm
- net N$26: track 72.5 -> 62.2 mm
- net N$29: track 55.4 -> 60.5 mm, vias 0 -> 1
- net N$28: track 56.3 -> 59.2 mm
- net N$25: track 53.8 -> 55.4 mm
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- added copper zone on layer 16, net GND
- added copper zone on layer 1, net N$32
Other:
- board text added: "Model M USB Controller Tygr Labs v1.0"
